Commit message: fix gripper

File: mycobot_gazebo/urdf/mycobot_280_ros2_control.xacro (robot description, xacro)
@@ -55,11 +55,7 @@
             <state_interface name="velocity"/>
         </joint>
-        <!-- <joint name="gripper_base_to_gripper_left2">
+        <joint name="gripper_base_to_gripper_left2">
             <param name="mimic">gripper_controller</param>
             <param name="multiplier">1.0</param>
-            <command_interface name="position">
-                <param name="min">-0.8</param>
-                <param name="max">0.5</param>
-            </command_interface>
             <state_interface name="position"/>
             <state_interface name="velocity"/>
@@ -68,8 +64,4 @@
             <param name="mimic">gripper_controller</param>
             <param name="multiplier">-1.0</param>
-            <command_interface name="position">
-                <param name="min">-0.5</param>
-                <param name="max">0.5</param>
-            </command_interface>
             <state_interface name="position"/>
             <state_interface name="velocity"/>
@@ -78,8 +70,4 @@
             <param name="mimic">gripper_controller</param>
             <param name="multiplier">-1.0</param>
-            <command_interface name="position">
-                <param name="min">-0.15</param>
-                <param name="max">0.7</param>
-            </command_interface>
             <state_interface name="position"/>
             <state_interface name="velocity"/>
@@ -88,8 +76,4 @@
             <param name="mimic">gripper_controller</param>
             <param name="multiplier">-1.0</param>
-            <command_interface name="position">
-                <param name="min">-0.5</param>
-                <param name="max">0.8</param>
-            </command_interface>
             <state_interface name="position"/>
             <state_interface name="velocity"/>
@@ -98,11 +82,7 @@
             <param name="mimic">gripper_controller</param>
             <param name="multiplier">1.0</param>
-            <command_interface name="position">
-                <param name="min">-0.5</param>
-                <param name="max">0.5</param>
-            </command_interface>
             <state_interface name="position"/>
             <state_interface name="velocity"/>
-        </joint> -->
+        </joint>
     </ros2_control>
 </robot>
